File: switch.kicad_sch (KiCad schematic)
At the start: 2 parts, among them SW1 KMR231NG

Commit message: Added LSCS part numbers to all components
Parts:
- R17: LCSC (none) -> C25900
- SW1: LCSC (none) -> C221680
Changed lines of the file:
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@@
+			)
+		)
+		(property "LCSC" "C25900"
+			(at 135.89 81.28 0)
+			(effects
+				(font
+					(size 1.27 1.27)
+				)
+				(hide yes)
 			)
 		)
@@
 			(effects
 				(font
+					(size 1.27 1.27)
+				)
+				(hide yes)
+			)
+		)
+		(property "LCSC" "C221680"
+			(at 135.89 93.98 90)
+			(effects
+				(font
