File: LED Breakout.kicad_pcb (KiCad board)
At the start: 2 copper layers, 32.5 x 27.7 mm, 41 parts, among them J1 Conn_02x10_Odd_Even, Q1 MMBT3904, Q2 MMBT3904, Q3 MMBT3904, Q4 MMBT3904, Q5 MMBT3904, Q6 MMBT3904, Q7 MMBT3904, Q8 MMBT3904, SW1 KMR231NG, SW2 KMR231NG, SW3 KMR231NG, SW4 KMR231NG

Commit message: Implement ERC/DRC parser in kicad2xunit.py
  - Add comprehensive parsing logic for KiBot ERC/DRC output format
  - Extract issue types, severity levels, locations, and component context
  - Fix xUnitGenerator to use correct ERCIssue attributes
  - Support both WARNING and ERROR severity levels
  - Generate proper xUnit XML with detailed failure information for CI/CD integration

  🤖 Generated with [Claude Code](https://claude.ai/code)

  Co-Authored-By: Claude <noreply@anthropic.com>

  This commit message:
  - Starts with a clear action verb ("Implement")
  - Summarizes the main functionality added
  - Lists the key technical improvements
  - Mentions the CI/CD integration purpose
  - Follows the repository's commit style based on recent commits
Routing:
- net /IOB_5B: track 34.8 -> 26.5 mm
Changed lines of the file:
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@@
-	)
-	(segment
-		(start 86.4108 50.8)
-		(end 94.742 50.8)
-		(width 0.2)
-		(layer "F.Cu")
-		(net 10)
 	)
 	(segment
